File: Drone_Controller.kicad_sch (KiCad schematic)
At the start: 31 parts, among them J1 Conn_01x05_Pin, J2 Conn_01x05_Pin, J3 Conn_02x04_Odd_Even, J4 Conn_ST_STDC14, J6 USB_B_Micro, SW1 SW_Push_Dual_x2, SW2 SW_Push_Dual_x2, SW3 SW_Push_Dual_x2, SW4 SW_Push_Dual_x2, U1 STM32L476RGTx, U2 TP4057, U3 TC1262-3.3VDB

Commit message: Add files via upload
Parts:
- removed R1: 10K, symbol Device:R_Small
- removed SW1, SW2, SW3, SW4: SW_Push_Dual_x2, symbol Switch:SW_Push_Dual_x2
- removed U3: TC1262-3.3VDB, TC1262-3.3VDB:SOT-223-3, symbol TC1262-3.3VDB:TC1262-3.3VDB
- added C10, C12: 0.1uF, Capacitor_SMD:C_0603_1608Metric_Pad1.08x0.95mm_HandSolder, symbol Device:C_Small
- added C11: C_Small, Capacitor_SMD:C_0603_1608Metric_Pad1.08x0.95mm_HandSolder, symbol Device:C_Small
- added C13, C14, C15: 22uF, Capacitor_SMD:C_0603_1608Metric_Pad1.08x0.95mm_HandSolder, symbol Device:C_Small
- added C16: 10pF, Capacitor_SMD:C_0603_1608Metric_Pad1.08x0.95mm_HandSolder, symbol Device:C_Small
- added C17: 10uF, Capacitor_SMD:C_0603_1608Metric_Pad1.08x0.95mm_HandSolder, symbol Device:C_Small
- added J5, ToggleSwitch1: Conn_01x02_Socket, Connector_JST:JST_XH_B2B-XH-A_1x02_P2.50mm_Vertical, symbol Connector:Conn_01x02_Socket
- added J7, J8, J9: Conn_01x02_Socket, symbol Connector:Conn_01x02_Socket
- added L1: 1uH, Inductor_SMD:L_0805_2012Metric_Pad1.05x1.20mm_HandSolder, symbol Device:L_Small
- added R4, R6, R7: R_Small, Resistor_SMD:R_0603_1608Metric_Pad0.98x0.95mm_HandSolder, symbol Device:R_Small
- added R5: 100, Resistor_SMD:R_0603_1608Metric_Pad0.98x0.95mm_HandSolder, symbol Device:R_Small
- added R8: 1M, Resistor_SMD:R_0603_1608Metric_Pad0.98x0.95mm_HandSolder, symbol Device:R_Small
- added U3: TPS63060DSCR, Package_SON:Texas_DSC0010J, symbol TPS63060DSCR:TPS63060DSCR
- added U4: DW01A, Package_TO_SOT_SMD:SOT-23-6, symbol Battery_Management:DW01A
- added U5: 8205A, Package_TO_SOT_SMD:SOT-23-6, symbol 8205A:8205A
- C1, C2, C3, C4, C5, C6, C8, C9: footprint (none) -> Capacitor_SMD:C_0603_1608Metric_Pad1.08x0.95mm_HandSolder
- C7: value C_Small -> 10uF; footprint (none) -> Capacitor_SMD:C_0603_1608Metric_Pad1.08x0.95mm_HandSolder
- D1: footprint (none) -> Diode_SMD:D_SOD-123
- D2, D3: footprint (none) -> LED_SMD:LED_0603_1608Metric_Pad1.05x0.95mm_HandSolder
- H1, H2, H3, H4: footprint (none) -> MountingHole:MountingHole_3.2mm_M3_DIN965_Pad
- J1, J2: footprint (none) -> Connector_JST:JST_XH_B5B-XH-A_1x05_P2.50mm_Vertical
- J3: footprint (none) -> Connector_JST:JST_PHD_B8B-PHDSS_2x04_P2.00mm_Vertical
- J4: footprint Connector_PinHeader_1.27mm:PinHeader_2x07_P1.27mm_Horizontal -> Connector_PinHeader_1.27mm:PinHeader_2x07_P1.27mm_Vertical_SMD
- J6: footprint (none) -> Connector_USB:USB_Micro-B_Molex-105017-0001
- R2, R3: footprint (none) -> Resistor_SMD:R_0603_1608Metric_Pad0.98x0.95mm_HandSolder
- U2: footprint TP4057:SOT26 -> Package_TO_SOT_SMD:TSOT-23-6_HandSoldering
Connections:
- net +3.3V: now also C13.1, C14.1, C15.1, R6.1, R8.2, U3.9 (VOUT); no longer C1.2, C2.2, C3.2, C4.2, C5.1, C6.2, C7.1, C7.2, C8.1, C9.1, H1.1, H2.1, H3.1, H4.1, J1.2 (Pin_2), J2.2 (Pin_2), J3.1 (Pin_1), J4.11 (GNDDetect), J4.5 (GND), J4.7 (GND), J6.5 (GND), J6.6 (Shield), R3.1, U1.12 (VSSA), U1.18 (VSS), U1.31 (VSS), U1.47 (VSS), U1.63 (VSS), U2.2 (GND)
- net Button1: now also J7.1 (Pin_1)
- net Button2: now also J8.1 (Pin_1)
- net Button3: now also J9.1 (Pin_1)
- net RF_MOSI: now also U1.53 (PC12)
- net GND: now reaches U1.60 (BOOT0)
- net GND: now also C1.2, C2.2, C3.2, C4.2, C5.1, C6.2, C7.2, C8.1, C9.1, H1.1, H2.1, H3.1, H4.1, J1.2 (Pin_2), J2.2 (Pin_2), J3.1 (Pin_1), J4.11 (GNDDetect), J4.5 (GND), J4.7 (GND), J6.5 (GND), J6.6 (Shield), R3.1, U1.12 (VSSA), U1.18 (VSS), U1.31 (VSS), U1.47 (VSS), U1.63 (VSS), U2.2 (GND), C11.1, C12.2, C13.2, C14.2, C15.2, C16.2, C17.2, J7.2 (Pin_2), J8.2 (Pin_2), J9.2 (Pin_2), R4.2, R7.2, U3.11_1 (EP), U3.11_10 (EP), U3.11_11 (EP), U3.11_12 (EP), U3.11_13 (EP), U3.11_14 (EP), U3.11_2 (EP), U3.11_3 (EP), U3.11_4 (EP), U3.11_5 (EP), U3.11_6 (EP), U3.11_7 (EP), U3.11_8 (EP), U3.11_9 (EP), U3.4 (PS/SYNC), U3.7 (GND), U5.3
- net +BATT renamed BAT+
- net BAT+: now also C7.1, C11.2, C17.1, J5.2 (Pin_2), R5.2, U3.2 (VIN), U3.3 (EN)
- new net: C12.1, U3.6 (VAUX)
- new net: U5.2, U5.5
- new net: U4.3 (OC), U5.4
- new net: U4.1 (OD), U5.6
- new net: R4.1, U4.2 (CS)
- new net: C10.1, R5.1, U4.5 (VCC)
- new net: L1.1, U3.10 (L2)
- new net: L1.2, U3.1 (L1)
- new net: R8.1, U3.5 (PG)
- new net: J5.1 (Pin_1), ToggleSwitch1.2 (Pin_2)
- new net BAT-: C10.2, ToggleSwitch1.1 (Pin_1), U4.6 (GND), U5.1
- new net FB: C16.1, R6.2, R7.1, U3.8 (FB)
Other:
- note added: "Connecteur batterie"
- note added: "Module de charge"
- note added: "Régulateur de tension(TPS63060DSCR)"
- note removed: "TC1262 (LDO)"
- note removed: "TP4057"
- moved on the sheet: C5, D1, D2, D3, J6, R2, R3, U2
