File: Drone_Controller.kicad_pcb (KiCad board)
At the start: 2 copper layers, 60 x 53 mm, 47 parts, among them J1 Conn_01x05_Pin, J2 Conn_01x05_Pin, U2 TP4057, U3 TPS63060DSCR, U4 DW01A, U5 8205A

Commit message: Add files via upload
Routing:
- net USART_TX: track 20.5 -> 21.8 mm
- net GND: vias 7 -> 8
Other:
- board text added: "B"
- board text added: "D.Ma"
- board text added: "T"
